File: Chimera/Chimera/MCU.kicad_sch (KiCad schematic)
At the start: 32 parts, among them J10 DM3CS-SF, J8 Button, J9 USB_B_Micro, U3 RP2040, U8 W25Q128JVSIQ, X1 ABM8-272-T3

Commit message: Rewiring M2 and moved Debugging LEDS
Parts:
- added C8: .1uF, Capacitor_SMD:C_0805_2012Metric, symbol Device:C
- added J11: Reciver, Connector_JST:JST_SH_SM06B-SRSS-TB_1x06-1MP_P1.00mm_Horizontal, symbol Connector:Conn_01x06_Socket
- added R14, R42: 10k, Resistor_SMD:R_0805_2012Metric, symbol Device:R
- added R43, R44: 500k, Resistor_SMD:R_0805_2012Metric, symbol Device:R
- added R8: 100m, Resistor_SMD:R_0805_2012Metric, symbol Device:R
- added U9: OpAmp, chimera:SC70-5_LT_MCH-M, symbol OEM:OpAmp
Connections:
- net +3.3V: now also C8.2, U9.5 (V+)
- net GND: now also C8.1, J11.1 (Pin_1), R14.2, R43.1, R8.2, U9.2 (V-)
- net Transmitter-MCU_TX: now reaches U3.31 (GPIO20)
- net Transmitter-MCU_TX: now also J11.6 (Pin_6)
- net Transmitter-MCU_RX: now reaches U3.32 (GPIO21)
- net Transmitter-MCU_RX: now also J11.5 (Pin_5)
- new net: R42.1, R43.2, U9.1 (+)
- new net +5V: J11.2 (Pin_2)
- new net Current_Sense: R44.1, U9.4
- new net OpF-: R14.1, R44.2, U9.3 (-)
- new net Servo_Current_Sense: R42.2, R8.1
